File: electronics/coil_winder.kicad_sch (KiCad schematic)
At the start: 27 parts, among them M1 screw motor, M2 coil motor, SW1 L_BTN, SW2 R_BTN, SW3 U_BTN, SW4 W_BTN, SW5 HOMING_BTN, U1 coil motor driver, U2 screw motor driver

Commit message: v1
Parts:
- added C4, C5: 100nF 100V, symbol Device:C
- added C6: 68nF, symbol Device:C
- added C7: 1uF, symbol Device:C_Polarized
- added D5: 1N4148, symbol Device:D
- added L1: L unknown, symbol Device:L
- added LM393: (no value), symbol driver:lm393
- added Q1: PMOS irf9z34n, symbol Simulation_SPICE:PMOS
- added Q2: NPN N2222A, Package_TO_SOT_THT:TO-92_Inline, symbol Transistor_BJT:PN2222A
- added R10: 500, symbol Device:R
- added R11: 100 0.5W, symbol Device:R
- added R12, R13, R14: 10k, symbol Device:R
- added R15: 4k7, symbol Device:R
- added R8: 1k, symbol Device:R
- added R9: 47k, symbol Device:R
Connections:
- net +12V: now also C6.2, LM393. (GND), Q1.3 (S), R10.1, R12.1
- net +3.3V: now also R15.1
- net GND: now also C4.2, C6.1, C7.2, L1.2, LM393. (GND), Q2.1 (E), R13.2, R9.2
- new net: C5.1, LM393. (GND), R14.1
- new net: C7.1, LM393. (GND), R12.2, R13.1, R14.2
- new net: Q1.1 (D), R11.1
- new net: D5.2 (A), R11.2
- new net: C4.1, C5.2, D5.1 (K), L1.1
- new net: Q2.2 (B), R8.2, R9.1
- new net: Q1.2 (G), Q2.3 (C), R10.2
- new net GP8: R8.1
- new net GP9: LM393. (GND), R15.2
Other:
- note added: "Configure max current driver pot to ~0.8V"
- note added: "Configure max current driver pot to ~1.3V"
- note added: "Inductance meter circuitry"
